File: PCB/ledW.kicad_sch (KiCad schematic)
At the start: 8 parts, among them Q41 Q_NPN_BCE

Commit message: made some Changes
Parts:
- removed R43: 1k, Resistor_SMD:R_1206_3216Metric_Pad1.30x1.75mm_HandSolder, symbol Device:R
Connections:
- net LEDW: now also Q41.1 (B)
Changed lines of the file:
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@@
     (stroke (width 0) (type default) (color 0 0 0 0))
   )
-  (hierarchical_label "LEDW" (shape input) (at 133.35 101.6 180)
+  (hierarchical_label "LEDW" (shape input) (at 140.97 101.6 180)
     (effects (font (size 1.27 1.27)) (justify right))
   )
@@
       (effects (font (size 1.27 1.27)) hide)
     )
-    (pin "1")
-    (pin "2")
-  )
-  (symbol (lib_id "Device:R") (at 137.16 101.6 90) (unit 1)
-    (in_bom yes) (on_board yes) (fields_autoplaced)
-    (property "Reference" "R43" (id 0) (at 137.16 95.25 90))
-    (property "Value" "1k" (id 1) (at 137.16 97.79 90))
-    (property "Footprint" "Resistor_SMD:R_1206_3216Metric_Pad1.30x1.75mm_HandSolder" (id 2) (at 137.16 103.378 90)
-      (effects (font (size 1.27 1.27)) hide)
-    )
-    (property "Datasheet" "~" (id 3) (at 137.16 101.6 0)
-      (effects (font (size 1.27 1.27)) hide)
-    )
-    (property "Price" "0.0021" (id 4) (at 137.16 101.6 0)
-      (effects (font (size 1.27 1.27)) hide)
-    )
